Commit message: modified:   build/gg_bot/colcon_command_prefix_build.sh.env 	modified:   build/gg_bot/symlink_install_manifest.txt 	new file:   install/gg_bot/share/gg_bot/launch/__pycache__/launch_robot.launch.cpython-310.pyc 	new file:   install/gg_bot/share/gg_bot/launch/launch_robot.launch.py 	new file:   log/build_2026-03-14_01-48-59/events.log 	new file:   log/build_2026-03-14_01-48-59/gg_bot/command.log 	new file:   log/build_2026-03-14_01-48-59/gg_bot/stderr.log 	new file:   log/build_2026-03-14_01-48-59/gg_bot/stdout.log 	new file:   log/build_2026-03-14_01-48-59/gg_bot/stdout_stderr.log 	new file:   log/build_2026-03-14_01-48-59/gg_bot/streams.log 	new file:   log/build_2026-03-14_01-48-59/logger_all.log 	new file:   log/build_2026-03-14_01-51-01/events.log 	new file:   log/build_2026-03-14_01-51-01/gg_bot/command.log 	new file:   log/build_2026-03-14_01-51-01/gg_bot/stderr.log 	new file:   log/build_2026-03-14_01-51-01/gg_bot/stdout.log 	new file:   log/build_2026-03-14_01-51-01/gg_bot/stdout_stderr.log 	new file:   log/build_2026-03-14_01-51-01/gg_bot/streams.log 	new file:   log/build_2026-03-14_01-51-01/logger_all.log 	modified:   log/latest_build 	modified:   src/gg_bot/config/my_controllers.yaml 	modified:   src/gg_bot/description/ros2_control.xacro 	new file:   src/gg_bot/launch/launch_robot.launch.py

File: src/gg_bot/description/ros2_control.xacro (robot description, xacro)
@@ -1,28 +1,61 @@
 <?xml version="1.0"?>
 <robot xmlns:xacro="http://www.ros.org/wiki/xacro">
-    <ros2_control name="GazeboSystem" type="system">
-        <hardware>
-            <plugin>gazebo_ros2_control/GazeboSystem</plugin>
-        </hardware>
-        <joint name="left_wheel_joint">
-            <command_interface name="velocity">
-                <param name="min">-10</param>
-                <param name="max">10</param>
-            </command_interface>
-            <state_interface name="velocity"/>
-            <state_interface name="position"/>
-        </joint>
-        <joint name="right_wheel_joint">
-            <command_interface name="velocity">
-                <param name="min">-10</param>
-                <param name="max">10</param>
-            </command_interface>
-            <state_interface name="velocity"/>
-            <state_interface name="position"/>
-        </joint>
-    </ros2_control>
+    <xacro:unless value="$(arg sim_mode)">
+        <ros2_control name="RealRobot" type="system">
+            <hardware>
+                <plugin>diffdrive_arduino/DiffDriveArduino</plugin>
+                <param name="left_wheel_name">left_wheel_joint</param>
+                <param name="right_wheel_name">right_wheel_joint</param>
+                <param name="loop_rate">30</param>
+                <param name="device">/dev/ttyUSB0</param>
+                <param name="baud_rate">57600</param>
+                <param name="timeout">1000</param>
+                <param name="enc_counts_per_rev">3436</param>
+            </hardware>
+            <joint name="left_wheel_joint">
+                <command_interface name="velocity">
+                    <param name="min">-10</param>
+                    <param name="max">10</param>
+                </command_interface>
+                <state_interface name="velocity"/>
+                <state_interface name="position"/>
+            </joint>
+            <joint name="right_wheel_joint">
+                <command_interface name="velocity">
+                    <param name="min">-10</param>
+                    <param name="max">10</param>
+                </command_interface>
+                <state_interface name="velocity"/>
+                <state_interface name="position"/>
+            </joint>
+        </ros2_control>
+    </xacro:unless>
+    <xacro:if value="$(arg sim_mode)">
+        <ros2_control name="GazeboSystem" type="system">
+            <hardware>
+                <plugin>gazebo_ros2_control/GazeboSystem</plugin>
+            </hardware>
+            <joint name="left_wheel_joint">
+                <command_interface name="velocity">
+                    <param name="min">-10</param>
+                    <param name="max">10</param>
+                </command_interface>
+                <state_interface name="velocity"/>
+                <state_interface name="position"/>
+            </joint>
+            <joint name="right_wheel_joint">
+                <command_interface name="velocity">
+                    <param name="min">-10</param>
+                    <param name="max">10</param>
+                </command_interface>
+                <state_interface name="velocity"/>
+                <state_interface name="position"/>
+            </joint>
+        </ros2_control>
+    </xacro:if>
     <gazebo>
         <plugin name="gazebo_ros2_control" filename="libgazebo_ros2_control.so">
             <parameters>$(find gg_bot)/config/my_controllers.yaml</parameters>
+            <parameters>$(find gg_bot)/config/gaz_ros2_ctl_use_sim.yaml</parameters>
         </plugin>
     </gazebo>
